Commit message: Fix robot stability, imitation learning data collection, and IL world

File: src/robot_description/urdf/base/base.urdf.xacro (robot description, xacro)
@@ -21,5 +21,5 @@
 	  <inertial>
 		  <origin xyz="0 0 0"/>
-		  <mass value="1.167"/>
+		  <mass value="8.0"/>
 		<inertia ixx="0.0016" ixy="0" ixz="0" iyy="0.0016" iyz="0" izz="0.0032" />
 	  </inertial>

File: src/robot_description/urdf/elbow/elbow.xacro (robot description, xacro)
@@ -23,5 +23,5 @@
 	  <inertial>
 		<origin xyz="0.1079630000 0.0001158760 0"/>
-		<mass value="0.234589"/>
+		<mass value="0.05"/>
 		<inertia ixx="0.00003971" ixy="0.0000023528" ixz="0.0" iyy="0.0008878" iyz="0.0" izz="0.000888"/>
 	  </inertial>

File: src/robot_description/urdf/finger/finger.xacro (robot description, xacro)
@@ -23,5 +23,5 @@
 	  <inertial>
 		<origin xyz="0.0 0.0 0.0"/>
-		<mass value="0.016"/>
+		<mass value="0.01"/>
 		<inertia ixx="0.000004731" ixy="-0.000000456" ixz="0.0" iyy="0.000003500" iyz="0.0" izz="0.000003747"/>
 	  </inertial>

File: src/robot_description/urdf/gripper/gripper.xacro (robot description, xacro)
@@ -23,5 +23,5 @@
 	  <inertial>
 		<origin xyz="0.0 0.0 0.0"/>
-		<mass value="0.25"/>
+		<mass value="0.03"/>
 		<inertia ixx="0.00002537" ixy="0.0" ixz="0.0" iyy="0.00001836" iyz="0.000000434" izz="0.00001674"/>
 	  </inertial>

File: src/robot_description/urdf/lower_arm/lower_arm.xacro (robot description, xacro)
@@ -23,5 +23,5 @@
 	  <inertial>
 		<origin xyz="0.0374395000 0.0052225200 0"/>
-		<mass value="0.220991"/>
+		<mass value="0.05"/>
 		<inertia ixx="0.00006369" ixy="-0.00002292" ixz="0.0" iyy="0.0001677" iyz="0.0" izz="0.0001834"/>
 	  </inertial>

File: src/robot_description/urdf/ros2_control.xacro (robot description, xacro)
@@ -53,4 +53,5 @@
       <joint_name>left_wheel_joint</joint_name>
       <joint_name>right_wheel_joint</joint_name>
+      <!-- casters are fixed joints — no joint states needed -->
       <joint_name>soulder_joint</joint_name>
       <joint_name>upper_arm_joint</joint_name>

File: src/robot_description/urdf/shoulder/shoulder.xacro (robot description, xacro)
@@ -23,5 +23,5 @@
 	  <inertial>
 		<origin xyz="0.0000223482 0.0000414609 0.0066287000"/>
-		<mass value="0.480879"/>
+		<mass value="0.05"/>
 		<inertia ixx="0.000222" ixy="0" ixz="0" iyy="0.000395" iyz="0" izz="0.000222"/>
 	  </inertial>

File: src/robot_description/urdf/upper_arm/upper_arm.xacro (robot description, xacro)
@@ -23,5 +23,5 @@
 	  <inertial>
 		<origin xyz="0.0 0.0 0.0"/>
-		<mass value="0.298"/>
+		<mass value="0.05"/>
 		<inertia ixx="0.002176" ixy="-0.0000030658" ixz="0.0" iyy="0.00005757" iyz="0.0" izz="0.002186"/>
 	  </inertial>

File: src/robot_description/urdf/wheels/diff_wheels.xacro (robot description, xacro)
@@ -1,83 +1,105 @@
 <?xml version="1.0"?>
 <robot xmlns:xacro="http://ros.org/wiki/xacro">
-  <!-- Differential drive wheels + caster + Gazebo diff_drive plugin -->
+  <!-- Differential drive: 2 driven wheels + 2 casters
+       All 4 placed at the same corner positions as the original omni wheels -->
   <xacro:macro name="diff_wheels_v0">
-    <!-- Left drive wheel -->
+    <!-- Left drive wheel — at the left-centre position (y=+0.086338) -->
     <joint name="left_wheel_joint" type="continuous">
       <parent link="base_link"/>
       <child link="left_wheel_link"/>
-      <origin xyz="0.0 0.175 0.0" rpy="-1.5707963 0 0"/>
+      <origin xyz="0.0 0.086338 -0.022" rpy="-1.5707963 0 0"/>
       <axis xyz="0 0 1"/>
     </joint>
     <link name="left_wheel_link">
       <visual>
-        <geometry><cylinder radius="0.05" length="0.04"/></geometry>
-        <material name="wheel_dark"><color rgba="0.15 0.15 0.15 1.0"/></material>
+        <geometry><cylinder radius="0.028" length="0.025"/></geometry>
+        <material name="wheel_dark"><color rgba="0.1 0.1 0.1 1.0"/></material>
       </visual>
       <collision>
-        <geometry><cylinder radius="0.05" length="0.04"/></geometry>
+        <geometry><cylinder radius="0.028" length="0.025"/></geometry>
       </collision>
-      <xacro:inertial_cylinder mass="0.2" length="0.04" radius="0.05">
+      <xacro:inertial_cylinder mass="0.1" length="0.025" radius="0.028">
         <origin xyz="0 0 0" rpy="0 0 0"/>
       </xacro:inertial_cylinder>
     </link>
-    <!-- Right drive wheel -->
+    <!-- Right drive wheel — at the right-centre position (y=-0.086338) -->
     <joint name="right_wheel_joint" type="continuous">
       <parent link="base_link"/>
       <child link="right_wheel_link"/>
-      <origin xyz="0.0 -0.175 0.0" rpy="-1.5707963 0 0"/>
+      <origin xyz="0.0 -0.086338 -0.022" rpy="-1.5707963 0 0"/>
       <axis xyz="0 0 1"/>
     </joint>
     <link name="right_wheel_link">
       <visual>
-        <geometry><cylinder radius="0.05" length="0.04"/></geometry>
-        <material name="wheel_dark"><color rgba="0.15 0.15 0.15 1.0"/></material>
+        <geometry><cylinder radius="0.028" length="0.025"/></geometry>
+        <material name="wheel_dark"><color rgba="0.1 0.1 0.1 1.0"/></material>
       </visual>
       <collision>
-        <geometry><cylinder radius="0.05" length="0.04"/></geometry>
+        <geometry><cylinder radius="0.028" length="0.025"/></geometry>
       </collision>
-      <xacro:inertial_cylinder mass="0.2" length="0.04" radius="0.05">
+      <xacro:inertial_cylinder mass="0.1" length="0.025" radius="0.028">
         <origin xyz="0 0 0" rpy="0 0 0"/>
       </xacro:inertial_cylinder>
     </link>
-    <!-- Rear caster wheel (arm is at the front, caster at back) -->
-    <joint name="caster_wheel_joint" type="fixed">
+    <!-- Front caster — at the front-centre position (x=+0.086338) -->
+    <joint name="front_caster_joint" type="fixed">
       <parent link="base_link"/>
-      <child link="caster_wheel_link"/>
-      <origin xyz="-0.1 0.0 -0.025" rpy="0 0 0"/>
+      <child link="front_caster_link"/>
+      <origin xyz="0.086338 0.0 -0.030" rpy="0 0 0"/>
     </joint>
-    <link name="caster_wheel_link">
+    <link name="front_caster_link">
       <visual>
-        <geometry><sphere radius="0.025"/></geometry>
-        <material name="caster_grey"><color rgba="0.7 0.7 0.7 1.0"/></material>
+        <geometry><sphere radius="0.020"/></geometry>
+        <material name="caster_grey"><color rgba="0.5 0.5 0.5 1.0"/></material>
       </visual>
       <collision>
-        <geometry><sphere radius="0.025"/></geometry>
+        <geometry><sphere radius="0.020"/></geometry>
       </collision>
       <inertial>
         <mass value="0.05"/>
-        <inertia ixx="0.000013" ixy="0" ixz="0"
-                 iyy="0.000013" iyz="0"
-                 izz="0.000013"/>
+        <inertia ixx="0.000004" ixy="0" ixz="0"
+                 iyy="0.000004" iyz="0"
+                 izz="0.000004"/>
       </inertial>
     </link>
-    <!-- Wheel friction properties -->
+    <!-- Rear caster — at the rear-centre position (x=-0.086338) -->
+    <joint name="rear_caster_joint" type="fixed">
+      <parent link="base_link"/>
+      <child link="rear_caster_link"/>
+      <origin xyz="-0.086338 0.0 -0.030" rpy="0 0 0"/>
+    </joint>
+    <link name="rear_caster_link">
+      <visual>
+        <geometry><sphere radius="0.020"/></geometry>
+        <material name="caster_grey"><color rgba="0.5 0.5 0.5 1.0"/></material>
+      </visual>
+      <collision>
+        <geometry><sphere radius="0.020"/></geometry>
+      </collision>
+      <inertial>
+        <mass value="0.05"/>
+        <inertia ixx="0.000004" ixy="0" ixz="0"
+                 iyy="0.000004" iyz="0"
+                 izz="0.000004"/>
+      </inertial>
+    </link>
+    <!-- Gazebo friction properties -->
     <gazebo reference="left_wheel_link">
       <material>Gazebo/DarkGrey</material>
-      <mu1>1.0</mu1>
-      <mu2>1.0</mu2>
+      <mu1>1.0</mu1><mu2>1.0</mu2>
     </gazebo>
     <gazebo reference="right_wheel_link">
       <material>Gazebo/DarkGrey</material>
-      <mu1>1.0</mu1>
-      <mu2>1.0</mu2>
+      <mu1>1.0</mu1><mu2>1.0</mu2>
     </gazebo>
-    <!-- Caster is frictionless so it swivels freely -->
-    <gazebo reference="caster_wheel_link">
+    <gazebo reference="front_caster_link">
       <material>Gazebo/Grey</material>
-      <mu1>0.001</mu1>
-      <mu2>0.001</mu2>
+      <mu1>0.001</mu1><mu2>0.001</mu2>
     </gazebo>
-    <!-- Differential drive Gazebo plugin -->
+    <gazebo reference="rear_caster_link">
+      <material>Gazebo/Grey</material>
+      <mu1>0.001</mu1><mu2>0.001</mu2>
+    </gazebo>
+    <!-- Differential drive plugin -->
     <gazebo>
       <plugin name="diff_drive" filename="libgazebo_ros_diff_drive.so">
@@ -88,6 +110,6 @@
         <left_joint>left_wheel_joint</left_joint>
         <right_joint>right_wheel_joint</right_joint>
-        <wheel_separation>0.35</wheel_separation>
-        <wheel_diameter>0.1</wheel_diameter>
+        <wheel_separation>0.172676</wheel_separation>
+        <wheel_diameter>0.056</wheel_diameter>
         <max_wheel_torque>200</max_wheel_torque>
         <max_wheel_acceleration>10.0</max_wheel_acceleration>
@@ -97,4 +119,5 @@
         <odometry_frame>odom</odometry_frame>
         <robot_base_frame>base_footprint</robot_base_frame>
+        <command_timeout>0.3</command_timeout>
       </plugin>
     </gazebo>

File: src/robot_description/urdf/wrist/wrist.xacro (robot description, xacro)
@@ -23,5 +23,5 @@
 	  <inertial>
 		<origin xyz="0.0 0.0 0.0"/>
-		<mass value="0.085"/>
+		<mass value="0.03"/>
 		<inertia ixx="0.00003082" ixy="0.0000000191" ixz="0.0000000023" iyy="0.00002822" iyz="0.0000025481" izz="0.00003152"/>
 	  </inertial>
